File: pb_power/pb_power.sch (KiCad schematic (older format))
At the start: 1 part

Commit message: Something something
Connections:
- net ESP_RESET renamed C_RESET
- net SLEEP_CTRL renamed SLP_CTL
Changed lines of the file:
@@
 LIBS:contrib
 LIBS:valves
+LIBS:pb_power-cache
 EELAYER 25 0
 EELAYER END
@@
 GPIO_7
 Text Label 1350 1900 2    60   ~ 0
-ESP_RESET
+C_RESET
 $Comp
 L GND #PWR?
@@
 	2200 1600 2000 1600
 Text Label 2500 1700 0    60   ~ 0
-SLEEP_CTRL
+SLP_CTL
 Wire Wire Line
 	2000 1700 2500 1700
